File: GD32E103CBT6/GD32E103CBT6.kicad_pcb (KiCad board)
At the start: 2 copper layers, 15 parts, among them J1 DBG, U1 GD32E103CBTx, Y1 16MHz

Commit message: Move things around a little bit
Parts:
- moved C3 0.95 mm to (129.2, 87.2)
- moved Y1 0.20 mm to (129.2, 90.0)
Routing:
- net /PD1: track 6.87 -> 4.86 mm
- net GND: track 23.2 -> 22.7 mm, vias 10 -> 11
