File: GD32E103CBT6/GD32E103CBT6.kicad_pcb (KiCad board)
At the start: 2 copper layers, 15 parts, among them J1 DBG, U1 GD32E103CBTx, Y1 16MHz

Commit message: update files to kicad 6
Other:
- net class Default removed
