File: NCV68261/NCV68261.kicad_sch (KiCad schematic)
At the start: 8 parts, among them Q1 SiR186LDP, Q2 SiR186LDP, U1 NCV68261

Commit message: use smaller fets
Parts:
- removed Q1, Q2: SiR186LDP, Package_SO:PowerPAK_SO-8_Single, symbol Transistor_FET:Si7141DP
- added Q1, Q2: DMT6007LFG-7, Package_SON:Diodes_PowerDI3333-8, symbol meansOfCircuitDesign:DMN22M5UFG
Connections:
- net V_{BUS}: now also Q1.1 (S), Q1.2 (S), Q1.3 (S)
- net V_{PROT}: now also Q2.1 (S), Q2.2 (S), Q2.3 (S)
- net at R1.1: now also Q1.4 (G)
- net at U1.1 (S): now also Q1.5 (D), Q2.5 (D)
- net at R1.2, R2.1, U1.2 (G): now also Q2.4 (G)
Changed lines of the file:
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@@
     (pin "2")
-  )
-  (symbol (lib_id "Transistor_FET:Si7141DP") (at 134.62 72.39 270) (mirror x) (unit 1)
-    (in_bom yes) (on_board yes) (fields_autoplaced)
-    (property "Reference" "Q1" (id 0) (at 134.62 62.23 90))
-    (property "Value" "SiR186LDP" (id 1) (at 134.62 64.77 90))
-    (property "Footprint" "Package_SO:PowerPAK_SO-8_Single" (id 2) (at 132.715 67.31 0)
-      (effects (font (size 1.27 1.27) italic) (justify left) hide)
-    )
-    (property "Datasheet" "https://www.vishay.com/docs/63001/sir186ldp.pdf" (id 3) (at 134.62 72.39 0)
-      (effects (font (size 1.27 1.27)) (justify left) hide)
-    )
-    (property "MPN" "SIR186LDP-T1-RE3" (id 4) (at 134.62 72.39 90)
-      (effects (font (size 1.27 1.27)) hide)
-    )
-    (pin "1")
-    (pin "2")
-    (pin "3")
-    (pin "4")
-    (pin "5")
   )
   (symbol (lib_id "power:GND") (at 161.29 77.47 0) (unit 1)
@@
     (pin "6")
   )
-  (symbol (lib_id "Transistor_FET:Si7141DP") (at 149.86 72.39 90) (unit 1)
-    (in_bom yes) (on_board yes) (fields_autoplaced)
-    (property "Reference" "Q2" (id 0) (at 149.86 62.23 90))
-    (property "Value" "SiR186LDP" (id 1) (at 149.86 64.77 90))
-    (property "Footprint" "Package_SO:PowerPAK_SO-8_Single" (id 2) (at 151.765 67.31 0)
-      (effects (font (size 1.27 1.27) italic) (justify left) hide)
-    )
-    (property "Datasheet" "https://www.vishay.com/docs/63001/sir186ldp.pdf" (id 3) (at 149.86 72.39 0)
-      (effects (font (size 1.27 1.27)) (justify left) hide)
-    )
-    (property "MPN" "SIR186LDP-T1-RE3" (id 4) (at 149.86 72.39 90)
-      (effects (font (size 1.27 1.27)) hide)
-    )
-    (pin "1")
-    (pin "2")
-    (pin "3")
-    (pin "4")
-    (pin "5")
-  )
   (symbol (lib_id "power:GND") (at 156.21 93.98 0) (unit 1)
     (in_bom yes) (on_board yes) (fields_autoplaced)
@@
     (pin "2")
   )
+  (symbol (lib_id "meansOfCircuitDesign:DMN22M5UFG") (at 149.86 72.39 90) (unit 1)
+    (in_bom yes) (on_board yes) (fields_autoplaced)
+    (property "Reference" "Q2" (id 0) (at 149.86 62.23 90))
+    (property "Value" "DMT6007LFG-7" (id 1) (at 149.86 64.77 90))
+    (property "Footprint" "Package_SON:Diodes_PowerDI3333-8" (id 2) (at 151.765 67.31 0)
+      (effects (font (size 1.27 1.27) italic) (justify left) hide)
+    )
+    (property "Datasheet" "https://www.diodes.com/assets/Datasheets/DMT6007LFG.pdf" (id 3) (at 149.86 72.39 90)
+      (effects (font (size 1.27 1.27)) (justify left) hide)
+    )
+    (property "MPN" "DMT6007LFG-7" (id 4) (at 149.86 72.39 0)
+      (effects (font (size 1.27 1.27)) hide)
+    )
+    (pin "1")
+    (pin "2")
+    (pin "3")
+    (pin "4")
+    (pin "5")
+  )
   (symbol (lib_id "Device:R_Small") (at 138.43 78.74 90) (unit 1)
     (in_bom yes) (on_board yes) (fields_autoplaced)
@@
     (pin "2")
   )
+  (symbol (lib_id "meansOfCircuitDesign:DMN22M5UFG") (at 134.62 72.39 270) (mirror x) (unit 1)
+    (in_bom yes) (on_board yes) (fields_autoplaced)
+    (property "Reference" "Q1" (id 0) (at 134.62 62.23 90))
+    (property "Value" "DMT6007LFG-7" (id 1) (at 134.62 64.77 90))
+    (property "Footprint" "Package_SON:Diodes_PowerDI3333-8" (id 2) (at 132.715 67.31 0)
+      (effects (font (size 1.27 1.27) italic) (justify left) hide)
+    )
+    (property "Datasheet" "https://www.diodes.com/assets/Datasheets/DMT6007LFG.pdf" (id 3) (at 134.62 72.39 90)
+      (effects (font (size 1.27 1.27)) (justify left) hide)
+    )
+    (property "MPN" "DMT6007LFG-7" (id 4) (at 134.62 72.39 0)
+      (effects (font (size 1.27 1.27)) hide)
+    )
+    (pin "1")
+    (pin "2")
+    (pin "3")
+    (pin "4")
+    (pin "5")
+  )
   (sheet_instances
     (path "/" (page "1"))
@@
       (reference "C3") (unit 1) (value "10uF/63V") (footprint "Capacitor_SMD:C_1210_3225Metric")
     )
-    (path "/2f52d062-4cea-47f4-8c9d-2310e204a239"
-      (reference "Q1") (unit 1) (value "SiR186LDP") (footprint "Package_SO:PowerPAK_SO-8_Single")
+    (path "/eef5a242-c1e5-4ffb-a46c-59acf6a11df5"
+      (reference "Q1") (unit 1) (value "DMT6007LFG-7") (footprint "Package_SON:Diodes_PowerDI3333-8")
     )
-    (path "/70f362ba-72bb-4286-98a6-a6f8639b2ff2"
-      (reference "Q2") (unit 1) (value "SiR186LDP") (footprint "Package_SO:PowerPAK_SO-8_Single")
+    (path "/8d8c5267-c6d8-44d0-92eb-46cf63342513"
+      (reference "Q2") (unit 1) (value "DMT6007LFG-7") (footprint "Package_SON:Diodes_PowerDI3333-8")
     )
     (path "/b2d19c93-ad1d-4a7a-9e3e-bf951d227f17"
