File: STM32F072CBU6/STM32F072CBU6.kicad_pcb (KiCad board)
At the start: 2 copper layers, 12 parts, among them J1 DBG, U1 STM32F072CBUx

Commit message: update files to kicad 6
Other:
- net class Default removed
