File: USB-C/USB-C.kicad_pcb (KiCad board)
At the start: 2 copper layers, 6 parts, among them J1 USB_C_Receptacle_USB2.0, U1 USBLC6-2SC6

Commit message: update files to kicad 6
Other:
- net class Default removed
